Commit message: Fix default head position and orientation

File: urdf/calibration/calibration_constants.urdf.xacro (robot description, xacro)
@@ -11,7 +11,7 @@
   <xacro:include filename="$(find talos_description_calibration)/urdf/deg_to_rad.xacro" />
   <!--Constant parameters-->
-  <xacro:property name="camera_position_x" value="0.0" />
+  <xacro:property name="camera_position_x" value="0.066" />
   <xacro:property name="camera_position_y" value="0.0" />
-  <xacro:property name="camera_position_z" value="0.0" />
+  <xacro:property name="camera_position_z" value="0.1982" />
   <xacro:property name="camera_orientation_r" value="0.0" />
   <xacro:property name="camera_orientation_p" value="0.0" />
